File: main/main.kicad_sch (KiCad schematic)
At the start: 50 parts, among them J1 RJ45, J2 RJ45, J3 Connector, USB-TYPE-C-16P, J4 Conn_01x04_Pin, J5 Conn_01x04_Pin, Q1 MMBT3904, U2 2.4GHz

Commit message: Switched up GPIO to avoid strapping pins
Connections:
- net +3.3V: now also R7.1; no longer R7.2
- net BTN1: now also U2.6 (IO3); no longer U2.5 (IO2)
- net BTN2: now also U2.18 (IO4); no longer U2.6 (IO3)
- net BTN3: now also U2.19 (IO5); no longer U2.16 (IO10)
- net IO_INT: now also R7.2, U2.16 (IO10); no longer R7.1, U2.21 (IO7)
- no-connect marks 35 -> 38

Commit message: Started to layout PCB
Parts:
- J4, J5: footprint (none) -> Connector_PinHeader_2.54mm:PinHeader_1x04_P2.54mm_Vertical
Changed lines of the file:
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@@
 			)
 		)
-		(property "Footprint" ""
+		(property "Footprint" "Connector_PinHeader_2.54mm:PinHeader_1x04_P2.54mm_Vertical"
 			(at 81.28 119.38 0)
 			(hide yes)
@@
 			)
 		)
-		(property "Footprint" ""
+		(property "Footprint" "Connector_PinHeader_2.54mm:PinHeader_1x04_P2.54mm_Vertical"
 			(at 135.89 101.6 0)
 			(hide yes)

Commit message: PCB Progress
Parts:
- removed J5: Conn_01x04_Pin, Connector_PinHeader_2.54mm:PinHeader_1x04_P2.54mm_Vertical, symbol Connector:Conn_01x04_Pin
- added H1, H2, H3, H4: MountingHole, MountingHole:MountingHole_3.2mm_M3, symbol Mechanical:MountingHole
- added J6: Conn_01x08_Pin, Connector_PinHeader_2.54mm:PinHeader_1x08_P2.54mm_Vertical, symbol Connector:Conn_01x08_Pin
Connections:
- net +3.3V: now also J6.8 (Pin_8)
- net +5V: now also J6.2 (Pin_2)
- net EN: now also J6.5 (Pin_5)
- net GND: now also J6.1 (Pin_1), J6.7 (Pin_7)
- net SCK: now reaches U2.20 (IO6)
- net SCK: now also J6.3 (Pin_3)
- net MOSI: now reaches U2.21 (IO7)
- net MOSI: now also J6.4 (Pin_4)
- net DC: now reaches U2.5 (IO2)
- net DC: now also J6.6 (Pin_6)
- no-connect marks 38 -> 35
